Commit message: added missing suffix param

File: low_camera/_d435.urdf.xacro (robot description, xacro)
@@ -7,5 +7,5 @@
 -->
 <robot name="sensor_d435" xmlns:xacro="http://ros.org/wiki/xacro">
-  <xacro:macro name="sensor_d435" params="parent *origin">
+  <xacro:macro name="sensor_d435" params="parent suffix='' *origin">
     <xacro:property name="M_PI" value="3.1415926535897931" />
     <!-- The following values are approximate, and the camera node
@@ -26,20 +26,20 @@
     <xacro:property name="d435_cam_depth_py" value="0.0175"/>
     <xacro:property name="d435_cam_depth_pz" value="${d435_cam_height/2}"/>
-    <material name="aluminum">
+    <material name="aluminum${suffix}">
 	  <color rgba="0.5 0.5 0.5 1"/>
     </material>
     <!-- camera body, with origin at bottom screw mount -->
-    <joint name="camera_joint" type="fixed">
+    <joint name="camera_joint${suffix}" type="fixed">
       <xacro:insert_block name="origin" />
       <parent link="${parent}"/>
-      <child link="camera_bottom_screw_frame" />
+      <child link="camera_bottom_screw_frame${suffix}" />
     </joint>
-    <link name="camera_bottom_screw_frame"/>
-    <joint name="camera_link_joint" type="fixed">
+    <link name="camera_bottom_screw_frame${suffix}"/>
+    <joint name="camera_link_joint${suffix}" type="fixed">
       <origin xyz="0 ${d435_cam_depth_py} ${d435_cam_depth_pz}" rpy="0 0 0"/>
-      <parent link="camera_bottom_screw_frame"/>
-      <child link="camera_link" />
+      <parent link="camera_bottom_screw_frame${suffix}"/>
+      <child link="camera_link${suffix}" />
     </joint>
-    <link name="camera_link">
+    <link name="camera_link${suffix}">
       <visual>
       <origin xyz="${d435_cam_mount_from_center_offset} ${-d435_cam_depth_py} 0" rpy="${M_PI/2} 0 ${M_PI/2}"/>
@@ -49,5 +49,5 @@
           <!--<mesh filename="package://realsense2_camera/meshes/d435/d435.dae" />-->
         </geometry>
-        <material name="aluminum"/>
+        <material name="aluminum${suffix}"/>
       </visual>
       <collision>
@@ -65,55 +65,55 @@
     </link>
     <!-- camera depth joints and links -->
-    <joint name="camera_depth_joint" type="fixed">
+    <joint name="camera_depth_joint${suffix}" type="fixed">
       <origin xyz="0 0 0" rpy="0 0 0"/>
-      <parent link="camera_link"/>
-      <child link="camera_depth_frame" />
+      <parent link="camera_link${suffix}"/>
+      <child link="camera_depth_frame${suffix}" />
     </joint>
-    <link name="camera_depth_frame"/>
-    <joint name="camera_depth_optical_joint" type="fixed">
+    <link name="camera_depth_frame${suffix}"/>
+    <joint name="camera_depth_optical_joint${suffix}" type="fixed">
       <origin xyz="0 0 0" rpy="${-M_PI/2} 0 ${-M_PI/2}" />
-      <parent link="camera_depth_frame" />
-      <child link="camera_depth_optical_frame" />
+      <parent link="camera_depth_frame${suffix}" />
+      <child link="camera_depth_optical_frame${suffix}" />
     </joint>
-    <link name="camera_depth_optical_frame"/>
+    <link name="camera_depth_optical_frame${suffix}"/>
     <!-- camera left IR joints and links -->
-    <joint name="camera_left_ir_joint" type="fixed">
+    <joint name="camera_left_ir_joint${suffix}" type="fixed">
       <origin xyz="0 ${d435_cam_depth_to_left_ir_offset} 0" rpy="0 0 0" />
-      <parent link="camera_depth_frame" />
-      <child link="camera_left_ir_frame" />
+      <parent link="camera_depth_frame${suffix}" />
+      <child link="camera_left_ir_frame${suffix}" />
     </joint>
-    <link name="camera_left_ir_frame"/>
-    <joint name="camera_left_ir_optical_joint" type="fixed">
+    <link name="camera_left_ir_frame${suffix}"/>
+    <joint name="camera_left_ir_optical_joint${suffix}" type="fixed">
       <origin xyz="0 0 0" rpy="${-M_PI/2} 0 ${-M_PI/2}" />
-      <parent link="camera_left_ir_frame" />
-      <child link="camera_left_ir_optical_frame" />
+      <parent link="camera_left_ir_frame${suffix}" />
+      <child link="camera_left_ir_optical_frame${suffix}" />
     </joint>
-    <link name="camera_left_ir_optical_frame"/>
+    <link name="camera_left_ir_optical_frame${suffix}"/>
     <!-- camera right IR joints and links -->
-    <joint name="camera_right_ir_joint" type="fixed">
+    <joint name="camera_right_ir_joint${suffix}" type="fixed">
       <origin xyz="0 ${d435_cam_depth_to_right_ir_offset} 0" rpy="0 0 0" />
-      <parent link="camera_depth_frame" />
-      <child link="camera_right_ir_frame" />
+      <parent link="camera_depth_frame${suffix}" />
+      <child link="camera_right_ir_frame${suffix}" />
     </joint>
-    <link name="camera_right_ir_frame"/>
-    <joint name="camera_right_ir_optical_joint" type="fixed">
+    <link name="camera_right_ir_frame${suffix}"/>
+    <joint name="camera_right_ir_optical_joint${suffix}" type="fixed">
       <origin xyz="0 0 0" rpy="${-M_PI/2} 0 ${-M_PI/2}" />
-      <parent link="camera_right_ir_frame" />
-      <child link="camera_right_ir_optical_frame" />
+      <parent link="camera_right_ir_frame${suffix}" />
+      <child link="camera_right_ir_optical_frame${suffix}" />
     </joint>
-    <link name="camera_right_ir_optical_frame"/>
+    <link name="camera_right_ir_optical_frame${suffix}"/>
     <!-- camera color joints and links -->
-    <joint name="camera_color_joint" type="fixed">
+    <joint name="camera_color_joint${suffix}" type="fixed">
       <origin xyz="0 ${d435_cam_depth_to_color_offset} 0" rpy="0 0 0" />
-      <parent link="camera_depth_frame" />
-      <child link="camera_color_frame" />
+      <parent link="camera_depth_frame${suffix}" />
+      <child link="camera_color_frame${suffix}" />
     </joint>
-    <link name="camera_color_frame"/>
-    <joint name="camera_color_optical_joint" type="fixed">
+    <link name="camera_color_frame${suffix}"/>
+    <joint name="camera_color_optical_joint${suffix}" type="fixed">
       <origin xyz="0 0 0" rpy="${-M_PI/2} 0 ${-M_PI/2}" />
-      <parent link="camera_color_frame" />
-      <child link="camera_color_optical_frame" />
+      <parent link="camera_color_frame${suffix}" />
+      <child link="camera_color_optical_frame${suffix}" />
     </joint>
-    <link name="camera_color_optical_frame"/>
+    <link name="camera_color_optical_frame${suffix}"/>
   </xacro:macro>
 </robot>

File: low_description/urdf/low.urdf.xacro (robot description, xacro)
@@ -12,5 +12,5 @@
     <color rgba="0 0 0 1"/>
   </material>
-  <xacro:include filename="$(find realsense2_camera)/urdf/_d435.urdf.xacro" />
+  <xacro:include filename="../../low_camera/_d435.urdf.xacro" />
   <xacro:include filename="$(find uos_common_urdf)/common.xacro" />
   <xacro:include filename="$(find uos_common_urdf)/urdf/imu.gazebo.urdf.xacro" />
