Commit message: added velodyne sensor to urdf

File: low_description/urdf/low.urdf.xacro (robot description, xacro)
@@ -9,4 +9,5 @@
   <xacro:include filename="$(find uos_common_urdf)/urdf/imu.gazebo.urdf.xacro" />
   <xacro:include filename="$(find sick_tim)/urdf/sick_tim.urdf.xacro" />
+  <xacro:include filename="$(find velodyne_description)/urdf/VLP-16.urdf.xacro" />
   <xacro:property name="M_PI" value="3.14159265359"/>
   <xacro:property name="imu_stdev" value="0.00017" />
@@ -159,4 +160,12 @@
       rpy="${M_PI} 0 ${M_PI/2.0}" />
   </joint>
+  <xacro:VLP-16>
+    <origin xyz="0 0 0.205"/>
+  </xacro:VLP-16>
+ <joint name="VLP-16_joint" type="fixed">
+    <parent link="base_link" />
+    <child link="velodyne" />
+    <child link="velodyne_base_link" />
+  </joint>
   <!-- inertial measurement unit for gazebo -->
   <xacro:imu_gazebo link="imu" imu_topic="imu/data" update_rate="100.0" stdev="${imu_stdev}" />

Commit message: debug

File: low_description/urdf/low.urdf.xacro (robot description, xacro)
@@ -12,6 +12,7 @@
   <xacro:property name="M_PI" value="3.14159265359"/>
   <xacro:property name="imu_stdev" value="0.00017" />
-  <xacro:property name="body_height" value="0.15"/>
-  <xacro:property name="body_length" value="0.48"/>
+  <!-- 0.48 -->
+  <xacro:property name="body_height" value="0.2"/>
+  <xacro:property name="body_length" value="0.8"/>
   <xacro:property name="body_width" value="0.32"/>
   <xacro:property name="axis_front" value="0.16"/>
@@ -163,9 +164,5 @@
     <origin xyz="0 0 0.205"/>
   </xacro:VLP-16>
- <joint name="VLP-16_joint" type="fixed">
-    <parent link="base_link" />
-    <child link="velodyne" />
-    <child link="velodyne_base_link" />
-  </joint>
+255
   <!-- inertial measurement unit for gazebo -->
   <xacro:imu_gazebo link="imu" imu_topic="imu/data" update_rate="100.0" stdev="${imu_stdev}" />

Commit message: added realsense to robot model (urdf)

File: low_description/urdf/low.urdf.xacro (robot description, xacro)
@@ -6,4 +6,11 @@
   xmlns:sensor="http://playerstage.sourceforge.net/gazebo/xmlschema/#sensor"
   name="low">
+  <material name="grey">
+    <color rgba="0.7 0 0 1"/>
+  </material>
+  <material name="black">
+    <color rgba="0 0 0 1"/>
+  </material>
+  <xacro:include filename="$(find realsense2_camera)/urdf/_d435.urdf.xacro" />
   <xacro:include filename="$(find uos_common_urdf)/common.xacro" />
   <xacro:include filename="$(find uos_common_urdf)/urdf/imu.gazebo.urdf.xacro" />
@@ -62,4 +69,15 @@
     <child link="base_link" />
   </joint>
+<!--Attach Realsense D435 Camera to robot-->
+  <xacro:sensor_d435
+    suffix="front"
+    parent="base_link">
+    <origin xyz="0.09 0 0.1625" rpy="0 0 0" />
+  </xacro:sensor_d435>
+  <!--xacro:sensor_d435
+    suffix="back"
+    parent="base_link">
+    <origin xyz="-0.325 0 0.085" rpy=" 0 0 ${M_PI}" />
+  </xacro:sensor_d435-->
   <!--Wheel Macro-->
   <xacro:macro name="wheel" params="name parent xyz side">

Commit message: combined velodyne and realsense, added gazebo support for both

File: low_description/urdf/low.urdf.xacro (robot description, xacro)
@@ -12,5 +12,8 @@
     <color rgba="0 0 0 1"/>
   </material>
-  <xacro:include filename="../../low_camera/_d435.urdf.xacro" />
+  <!--New Include D435-->
+  <xacro:include filename="$(find low_camera)/urdf/_d435.urdf.xacro" />
+  <!--New Include VLP-16-->
+  <xacro:include filename="$(find velodyne_description)/urdf/VLP-16.urdf.xacro"/>
   <xacro:include filename="$(find uos_common_urdf)/common.xacro" />
   <xacro:include filename="$(find uos_common_urdf)/urdf/imu.gazebo.urdf.xacro" />
@@ -80,4 +83,8 @@
     <origin xyz="-0.325 0 0.085" rpy=" 0 0 ${M_PI}" />
   </xacro:sensor_d435-->
+  <!--Attach VLP-16 to robot-->
+  <xacro:VLP-16>
+    <origin xyz="0 0 0.205"/>
+  </xacro:VLP-16>
   <!--Wheel Macro-->
   <xacro:macro name="wheel" params="name parent xyz side">

Commit message: changed spawn position of the robot

File: low_description/urdf/low.urdf.xacro (robot description, xacro)
@@ -23,5 +23,5 @@
   <xacro:property name="imu_stdev" value="0.00017" />
   <xacro:property name="body_height" value="0.2"/>
-  <xacro:property name="body_length" value="0.8"/>
+  <xacro:property name="body_length" value="0.48"/>
   <xacro:property name="body_width" value="0.32"/>
   <xacro:property name="axis_front" value="0.16"/>
