Commit message: added loal frames

File: acorn_description/urdf/acorn.urdf.xacro (robot description, xacro)
@@ -169,4 +169,18 @@
     <origin xyz="-${laser_x} 0 ${laser_z}" rpy="${M_PI} 0 ${M_PI}"/>
   </joint>
+  <!-- loal -->
+  <link name="camera_base"/>
+  <joint name="camera_base_joint" type="fixed">
+    <parent link="velodyne" />
+    <child link="camera_base" />
+    <origin xyz="0 0 0" rpy="0 0 0"/>
+  </joint>
+  <link name="camera"/>
+  <joint name="camera_joint" type="fixed">
+    <parent link="camera_base" />
+    <child link="camera" />
+    <origin xyz="0 0 0" rpy="1.570795 0 1.570795"/>
+  </joint>
+  <!-- loal end -->
   <link name="imu">
     <visual>

Commit message: move camera (for loal) to root of tf tree

File: acorn_description/urdf/acorn.urdf.xacro (robot description, xacro)
@@ -172,13 +172,13 @@
   <link name="camera_base"/>
   <joint name="camera_base_joint" type="fixed">
-    <parent link="velodyne" />
-    <child link="camera_base" />
-    <origin xyz="0 0 0" rpy="0 0 0"/>
+    <parent link="camera_base" />
+    <child link="base_footprint" />
+    <origin xyz="0 0 ${axis_height - wheel_radius - 0.205}" rpy="0 0 0"/>
   </joint>
   <link name="camera"/>
   <joint name="camera_joint" type="fixed">
-    <parent link="camera_base" />
-    <child link="camera" />
-    <origin xyz="0 0 0" rpy="1.570795 0 1.570795"/>
+    <parent link="camera" />
+    <child link="camera_base" />
+    <origin xyz="0 0 0" rpy="-1.570795 -1.570795 0"/>
   </joint>
   <!-- loal end -->
